Commit message: Renamed from <model>_<variant> to <model><variant>

File: fanuc_r2000ic_support/urdf/r2000ic125l_macro.xacro (robot description, xacro)
@@ -2,5 +2,5 @@
 <robot xmlns:xacro="http://ros.org/wiki/xacro">
   <xacro:include filename="$(find fanuc_resources)/urdf/common_materials.xacro"/>
-  <xacro:macro name="fanuc_r2000ic_125l" params="prefix">
+  <xacro:macro name="fanuc_r2000ic125l" params="prefix">
     <!-- link list -->
     <link name="${prefix}base_link">
@@ -8,5 +8,5 @@
         <origin xyz="0 0 0" rpy="0 0 0"/>
         <geometry>
-          <mesh filename="package://fanuc_r2000ic_support/meshes/r2000ic_125l/visual/base_link.stl"/>
+          <mesh filename="package://fanuc_r2000ic_support/meshes/r2000ic125l/visual/base_link.stl"/>
         </geometry>
         <xacro:material_fanuc_gray31 />
@@ -14,5 +14,5 @@
       <collision>
         <geometry>
-          <mesh filename="package://fanuc_r2000ic_support/meshes/r2000ic_125l/collision/base_link.stl"/>
+          <mesh filename="package://fanuc_r2000ic_support/meshes/r2000ic125l/collision/base_link.stl"/>
         </geometry>
         <xacro:material_fanuc_gray31 />
@@ -23,5 +23,5 @@
         <origin xyz="0 0 0" rpy="0 0 0"/>
         <geometry>
-          <mesh filename="package://fanuc_r2000ic_support/meshes/r2000ic_125l/visual/link_1.stl"/>
+          <mesh filename="package://fanuc_r2000ic_support/meshes/r2000ic125l/visual/link_1.stl"/>
         </geometry>
         <xacro:material_fanuc_yellow />
@@ -30,5 +30,5 @@
         <origin xyz="0 0 0" rpy="0 0 0"/>
         <geometry>
-          <mesh filename="package://fanuc_r2000ic_support/meshes/r2000ic_125l/collision/link_1.stl"/>
+          <mesh filename="package://fanuc_r2000ic_support/meshes/r2000ic125l/collision/link_1.stl"/>
         </geometry>
         <xacro:material_fanuc_yellow />
@@ -39,5 +39,5 @@
         <origin xyz="0 0 0" rpy="0 0 0"/>
         <geometry>
-          <mesh filename="package://fanuc_r2000ic_support/meshes/r2000ic_125l/visual/link_2.stl"/>
+          <mesh filename="package://fanuc_r2000ic_support/meshes/r2000ic125l/visual/link_2.stl"/>
         </geometry>
         <xacro:material_fanuc_yellow />
@@ -46,5 +46,5 @@
         <origin xyz="0 0 0" rpy="0 0 0"/>
         <geometry>
-          <mesh filename="package://fanuc_r2000ic_support/meshes/r2000ic_125l/collision/link_2.stl"/>
+          <mesh filename="package://fanuc_r2000ic_support/meshes/r2000ic125l/collision/link_2.stl"/>
         </geometry>
         <xacro:material_fanuc_yellow />
@@ -55,5 +55,5 @@
         <origin xyz="0 0 0" rpy="0 0 0"/>
         <geometry>
-          <mesh filename="package://fanuc_r2000ic_support/meshes/r2000ic_125l/visual/link_3.stl"/>
+          <mesh filename="package://fanuc_r2000ic_support/meshes/r2000ic125l/visual/link_3.stl"/>
         </geometry>
         <xacro:material_fanuc_yellow />
@@ -62,5 +62,5 @@
         <origin xyz="0 0 0" rpy="0 0 0"/>
         <geometry>
-          <mesh filename="package://fanuc_r2000ic_support/meshes/r2000ic_125l/collision/link_3.stl"/>
+          <mesh filename="package://fanuc_r2000ic_support/meshes/r2000ic125l/collision/link_3.stl"/>
         </geometry>
         <xacro:material_fanuc_yellow />
@@ -71,5 +71,5 @@
         <origin xyz="1.730 0 0" rpy="0 0 0"/>
         <geometry>
-          <mesh filename="package://fanuc_r2000ic_support/meshes/r2000ic_125l/visual/link_4.stl"/>
+          <mesh filename="package://fanuc_r2000ic_support/meshes/r2000ic125l/visual/link_4.stl"/>
         </geometry>
         <xacro:material_fanuc_yellow />
@@ -78,5 +78,5 @@
         <origin xyz="1.730 0 0" rpy="0 0 0"/>
         <geometry>
-          <mesh filename="package://fanuc_r2000ic_support/meshes/r2000ic_125l/collision/link_4.stl"/>
+          <mesh filename="package://fanuc_r2000ic_support/meshes/r2000ic125l/collision/link_4.stl"/>
         </geometry>
         <xacro:material_fanuc_yellow />
@@ -87,5 +87,5 @@
         <origin xyz="0 0 0" rpy="0 0 0"/>
         <geometry>
-          <mesh filename="package://fanuc_r2000ic_support/meshes/r2000ic_125l/visual/link_5.stl"/>
+          <mesh filename="package://fanuc_r2000ic_support/meshes/r2000ic125l/visual/link_5.stl"/>
         </geometry>
         <xacro:material_fanuc_yellow />
@@ -94,5 +94,5 @@
         <origin xyz="0 0 0" rpy="0 0 0"/>
         <geometry>
-          <mesh filename="package://fanuc_r2000ic_support/meshes/r2000ic_125l/collision/link_5.stl"/>
+          <mesh filename="package://fanuc_r2000ic_support/meshes/r2000ic125l/collision/link_5.stl"/>
         </geometry>
         <xacro:material_fanuc_yellow />
@@ -103,5 +103,5 @@
         <origin xyz="0 0 0" rpy="0 0 0"/>
         <geometry>
-          <mesh filename="package://fanuc_r2000ic_support/meshes/r2000ic_125l/visual/link_6.stl"/>
+          <mesh filename="package://fanuc_r2000ic_support/meshes/r2000ic125l/visual/link_6.stl"/>
         </geometry>
         <xacro:material_fanuc_black />
@@ -110,5 +110,5 @@
         <origin xyz="0 0 0" rpy="0 0 0"/>
         <geometry>
-          <mesh filename="package://fanuc_r2000ic_support/meshes/r2000ic_125l/collision/link_6.stl"/>
+          <mesh filename="package://fanuc_r2000ic_support/meshes/r2000ic125l/collision/link_6.stl"/>
         </geometry>
         <xacro:material_fanuc_black />

File: fanuc_r2000ic_support/urdf/r2000ic165f_macro.xacro (robot description, xacro)
@@ -2,5 +2,5 @@
 <robot xmlns:xacro="http://wiki.ros.org/xacro">
   <xacro:include filename="$(find fanuc_resources)/urdf/common_materials.xacro"/>
-  <xacro:macro name="fanuc_r2000ic_165f" params="prefix">
+  <xacro:macro name="fanuc_r2000ic165f" params="prefix">
     <!-- links: main serial chain -->
     <link name="${prefix}base_link">
@@ -8,5 +8,5 @@
         <origin xyz="0 0 0" rpy="0 0 0"/>
         <geometry>
-          <mesh filename="package://fanuc_r2000ic_support/meshes/r2000ic_165f/visual/base_link.stl"/>
+          <mesh filename="package://fanuc_r2000ic_support/meshes/r2000ic165f/visual/base_link.stl"/>
         </geometry>
         <xacro:material_fanuc_gray40 />
@@ -15,5 +15,5 @@
         <origin xyz="0 0 0" rpy="0 0 0"/>
         <geometry>
-          <mesh filename="package://fanuc_r2000ic_support/meshes/r2000ic_165f/collision/base_link.stl"/>
+          <mesh filename="package://fanuc_r2000ic_support/meshes/r2000ic165f/collision/base_link.stl"/>
         </geometry>
       </collision>
@@ -23,5 +23,5 @@
         <origin xyz="0 0 0" rpy="0 0 0"/>
         <geometry>
-          <mesh filename="package://fanuc_r2000ic_support/meshes/r2000ic_165f/visual/link_1.stl"/>
+          <mesh filename="package://fanuc_r2000ic_support/meshes/r2000ic165f/visual/link_1.stl"/>
         </geometry>
         <xacro:material_fanuc_yellow />
@@ -30,5 +30,5 @@
         <origin xyz="0 0 0" rpy="0 0 0"/>
         <geometry>
-          <mesh filename="package://fanuc_r2000ic_support/meshes/r2000ic_165f/collision/link_1.stl"/>
+          <mesh filename="package://fanuc_r2000ic_support/meshes/r2000ic165f/collision/link_1.stl"/>
         </geometry>
       </collision>
@@ -38,5 +38,5 @@
         <origin xyz="0 0 0" rpy="0 0 0"/>
         <geometry>
-          <mesh filename="package://fanuc_r2000ic_support/meshes/r2000ic_165f/visual/link_2.stl"/>
+          <mesh filename="package://fanuc_r2000ic_support/meshes/r2000ic165f/visual/link_2.stl"/>
         </geometry>
         <xacro:material_fanuc_yellow />
@@ -45,5 +45,5 @@
         <origin xyz="0 0 0" rpy="0 0 0"/>
         <geometry>
-          <mesh filename="package://fanuc_r2000ic_support/meshes/r2000ic_165f/collision/link_2.stl"/>
+          <mesh filename="package://fanuc_r2000ic_support/meshes/r2000ic165f/collision/link_2.stl"/>
         </geometry>
       </collision>
@@ -53,5 +53,5 @@
         <origin xyz="0 0 0" rpy="0 0 0"/>
         <geometry>
-          <mesh filename="package://fanuc_r2000ic_support/meshes/r2000ic_165f/visual/link_3.stl"/>
+          <mesh filename="package://fanuc_r2000ic_support/meshes/r2000ic165f/visual/link_3.stl"/>
         </geometry>
         <xacro:material_fanuc_yellow />
@@ -60,5 +60,5 @@
         <origin xyz="0 0 0" rpy="0 0 0"/>
         <geometry>
-          <mesh filename="package://fanuc_r2000ic_support/meshes/r2000ic_165f/collision/link_3.stl"/>
+          <mesh filename="package://fanuc_r2000ic_support/meshes/r2000ic165f/collision/link_3.stl"/>
         </geometry>
       </collision>
@@ -68,5 +68,5 @@
         <origin xyz="0 0 0" rpy="0 0 0"/>
         <geometry>
-          <mesh filename="package://fanuc_r2000ic_support/meshes/r2000ic_165f/visual/link_4.stl"/>
+          <mesh filename="package://fanuc_r2000ic_support/meshes/r2000ic165f/visual/link_4.stl"/>
         </geometry>
         <xacro:material_fanuc_yellow />
@@ -75,5 +75,5 @@
         <origin xyz="0 0 0" rpy="0 0 0"/>
         <geometry>
-          <mesh filename="package://fanuc_r2000ic_support/meshes/r2000ic_165f/collision/link_4.stl"/>
+          <mesh filename="package://fanuc_r2000ic_support/meshes/r2000ic165f/collision/link_4.stl"/>
         </geometry>
       </collision>
@@ -83,5 +83,5 @@
         <origin xyz="0 0 0" rpy="0 0 0"/>
         <geometry>
-          <mesh filename="package://fanuc_r2000ic_support/meshes/r2000ic_165f/visual/link_5.stl"/>
+          <mesh filename="package://fanuc_r2000ic_support/meshes/r2000ic165f/visual/link_5.stl"/>
         </geometry>
         <xacro:material_fanuc_yellow />
@@ -90,5 +90,5 @@
         <origin xyz="0 0 0" rpy="0 0 0"/>
         <geometry>
-          <mesh filename="package://fanuc_r2000ic_support/meshes/r2000ic_165f/collision/link_5.stl"/>
+          <mesh filename="package://fanuc_r2000ic_support/meshes/r2000ic165f/collision/link_5.stl"/>
         </geometry>
       </collision>
@@ -98,5 +98,5 @@
         <origin xyz="0 0 0" rpy="0 0 0"/>
         <geometry>
-          <mesh filename="package://fanuc_r2000ic_support/meshes/r2000ic_165f/visual/link_6.stl"/>
+          <mesh filename="package://fanuc_r2000ic_support/meshes/r2000ic165f/visual/link_6.stl"/>
         </geometry>
         <xacro:material_fanuc_black />
@@ -105,5 +105,5 @@
         <origin xyz="0 0 0" rpy="0 0 0"/>
         <geometry>
-          <mesh filename="package://fanuc_r2000ic_support/meshes/r2000ic_165f/collision/link_6.stl"/>
+          <mesh filename="package://fanuc_r2000ic_support/meshes/r2000ic165f/collision/link_6.stl"/>
         </geometry>
       </collision>
