Commit message: Reversed tool flange x-axis

File: fanuc_r2000ic_support/urdf/r2000ic165f_macro.xacro (robot description, xacro)
@@ -169,5 +169,5 @@
     <link name="${prefix}tool0" />
     <joint name="${prefix}link_6-tool0" type="fixed">
-      <origin xyz="0 0 0" rpy="${pi} ${-pi/2.0} 0" />
+      <origin xyz="0 0 0" rpy="0 ${radians(90)} 0" />
       <parent link="${prefix}link_6" />
       <child link="${prefix}tool0" />
